File: model_d/model_d.kicad_pcb (KiCad board)
At the start: 2 copper layers, 50 parts, among them J1 Conn_01x16_Male, J2 Conn_01x08_Male, SW1 SW_Cap, SW10 SW_Cap, SW11 SW_Cap, SW12 SW_Cap, SW13 SW_Cap, SW14 SW_Cap, SW15 SW_Cap, SW16 SW_Cap, SW17 SW_Cap, SW18 SW_Cap, SW19 SW_Cap, SW2 SW_Cap, SW20 SW_Cap, SW21 SW_Cap, SW22 SW_Cap, SW23 SW_Cap, SW24 SW_Cap, SW25 SW_Cap, SW26 SW_Cap, SW27 SW_Cap, SW28 SW_Cap, SW29 SW_Cap, SW3 SW_Cap, SW30 SW_Cap, SW31 SW_Cap, SW32 SW_Cap, SW33 SW_Cap, SW34 SW_Cap, SW35 SW_Cap, SW36 SW_Cap, SW37 SW_Cap, SW38 SW_Cap, SW39 SW_Cap, SW4 SW_Cap, SW40 SW_Cap, SW41 SW_Cap, SW42 SW_Cap, SW43 SW_Cap, SW44 SW_Cap, SW45 SW_Cap, SW46 SW_Cap, SW47 SW_Cap, SW48 SW_Cap, SW5 SW_Cap, SW6 SW_Cap, SW7 SW_Cap, SW8 SW_Cap, SW9 SW_Cap

Commit message: complete place & route, add gnd plate
Parts:
- removed J1: Conn_01x16_Male, Connector_PinHeader_2.54mm:PinHeader_1x16_P2.54mm_Vertical
- removed J2: Conn_01x08_Male, Connector_PinHeader_2.54mm:PinHeader_1x08_P2.54mm_Vertical
- added COL: Conn_01x27, Connector_PinHeader_2.54mm:PinHeader_1x27_P2.54mm_Vertical, F.Cu at (120.0, 36.0)
- added G***: LOGO, model_d:model_d, F.Cu at (42.5, 37.5)
- added ROW: Conn_01x12, Connector_PinHeader_2.54mm:PinHeader_1x12_P2.54mm_Vertical, F.Cu at (250.4, 32.4)
Routing:
- net GND: track 598.1 -> 1110.8 mm
- net C11: track 63.0 -> 175.4 mm
- net C0: track 77.2 -> 174.9 mm
- net C10: track 63.0 -> 160.4 mm
- net C1: track 63.0 -> 158.4 mm
- net C9: track 63.0 -> 144.2 mm
- net C2: track 63.0 -> 141.7 mm
- net C8: track 63.0 -> 128.0 mm
- net C3: track 68.2 -> 130.9 mm
- net C7: track 71.1 -> 119.3 mm
- net C4: track 63.0 -> 109.0 mm
- net C6: track 63.0 -> 94.5 mm
- net C5: track 63.0 -> 92.5 mm
- net R1: track 382.1 -> 407.8 mm
- net R0: track 376.2 -> 398.5 mm
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- added copper zone on B.Cu, net GND
- added copper zone on F.Cu, net GND
Other:
- board outline added: 244 x 105.5 mm
