File: model_d/model_d.kicad_pcb (KiCad board)
At the start: 2 copper layers, 244 x 105.5 mm, 51 parts, among them SW1 SW_Cap, SW10 SW_Cap, SW11 SW_Cap, SW12 SW_Cap, SW13 SW_Cap, SW14 SW_Cap, SW15 SW_Cap, SW16 SW_Cap, SW17 SW_Cap, SW18 SW_Cap, SW19 SW_Cap, SW2 SW_Cap, SW20 SW_Cap, SW21 SW_Cap, SW22 SW_Cap, SW23 SW_Cap, SW24 SW_Cap, SW25 SW_Cap, SW26 SW_Cap, SW27 SW_Cap, SW28 SW_Cap, SW29 SW_Cap, SW3 SW_Cap, SW30 SW_Cap, SW31 SW_Cap, SW32 SW_Cap, SW33 SW_Cap, SW34 SW_Cap, SW35 SW_Cap, SW36 SW_Cap, SW37 SW_Cap, SW38 SW_Cap, SW39 SW_Cap, SW4 SW_Cap, SW40 SW_Cap, SW41 SW_Cap, SW42 SW_Cap, SW43 SW_Cap, SW44 SW_Cap, SW45 SW_Cap, SW46 SW_Cap, SW47 SW_Cap, SW48 SW_Cap, SW5 SW_Cap, SW6 SW_Cap, SW7 SW_Cap, SW8 SW_Cap, SW9 SW_Cap

Commit message: add m3 mounting holes, increase size to 113x244
Parts:
- removed COL: Conn_01x27, Connector_PinHeader_2.54mm:PinHeader_1x27_P2.54mm_Vertical
- removed ROW: Conn_01x12, Connector_PinHeader_2.54mm:PinHeader_1x12_P2.54mm_Vertical
- added COLS: Conn_01x16, Connector_PinHeader_2.54mm:PinHeader_1x16_P2.54mm_Vertical, F.Cu at (120.0, 36.0)
- added REF**: MountingHole_3.2mm_M3, MountingHole:MountingHole_3.2mm_M3, F.Cu at (262.5, 30.0)
- added REF**: MountingHole_3.2mm_M3, MountingHole:MountingHole_3.2mm_M3, F.Cu at (183.8, 135.0)
- added REF**: MountingHole_3.2mm_M3, MountingHole:MountingHole_3.2mm_M3, F.Cu at (144.5, 135.0)
- added REF**: MountingHole_3.2mm_M3, MountingHole:MountingHole_3.2mm_M3, F.Cu at (105.2, 135.0)
- added REF**: MountingHole_3.2mm_M3, MountingHole:MountingHole_3.2mm_M3, F.Cu at (65.8, 135.0)
- added REF**: MountingHole_3.2mm_M3, MountingHole:MountingHole_3.2mm_M3, F.Cu at (26.5, 135.0)
- added REF**: MountingHole_3.2mm_M3, MountingHole:MountingHole_3.2mm_M3, F.Cu at (223.2, 30.0)
- added REF**: MountingHole_3.2mm_M3, MountingHole:MountingHole_3.2mm_M3, F.Cu at (183.8, 30.0)
- added REF**: MountingHole_3.2mm_M3, MountingHole:MountingHole_3.2mm_M3, F.Cu at (105.2, 30.0)
- added REF**: MountingHole_3.2mm_M3, MountingHole:MountingHole_3.2mm_M3, F.Cu at (65.8, 30.0)
- added REF**: MountingHole_3.2mm_M3, MountingHole:MountingHole_3.2mm_M3, F.Cu at (26.5, 30.0)
- added REF**: MountingHole_3.2mm_M3, MountingHole:MountingHole_3.2mm_M3, F.Cu at (144.5, 30.0)
- added REF**: MountingHole_3.2mm_M3, MountingHole:MountingHole_3.2mm_M3, F.Cu at (262.5, 135.0)
- added REF**: MountingHole_3.2mm_M3, MountingHole:MountingHole_3.2mm_M3, F.Cu at (223.2, 135.0)
- added ROWS: Conn_01x08, Connector_PinHeader_2.54mm:PinHeader_1x08_P2.54mm_Vertical, F.Cu at (263.0, 36.0)
Routing:
- net GND: track 1110.8 -> 1138.7 mm
- net R1: track 407.8 -> 390.5 mm
- net R0: track 398.5 -> 382.1 mm
- net R2: track 427.8 -> 411.7 mm
- net R3: track 449.3 -> 434.0 mm
Other:
- board size 244 x 105.5 mm -> 244 x 113 mm
