File: gndplate/_autosave-model_d.kicad_pcb (KiCad board)
At the start: 2 copper layers, 244 x 113 mm, 16 parts

Commit message: update gerbers
Parts:
- added G***: LOGO, model_d:model_d, B.Cu at (42.5, 37.5)
- added G***: LOGO, model_d:model_d, F.Cu at (42.5, 37.5)
