File: gndplate/model_d.kicad_pcb (KiCad board)
At the start: 2 copper layers, 244 x 105.5 mm, 2 parts

Commit message: add m3 mounting holes, increase size to 113x244
Parts:
- added REF**: MountingHole_3.2mm_M3, MountingHole:MountingHole_3.2mm_M3, F.Cu at (262.5, 30.0)
- added REF**: MountingHole_3.2mm_M3, MountingHole:MountingHole_3.2mm_M3, F.Cu at (26.5, 30.0)
- added REF**: MountingHole_3.2mm_M3, MountingHole:MountingHole_3.2mm_M3, F.Cu at (223.2, 30.0)
- added REF**: MountingHole_3.2mm_M3, MountingHole:MountingHole_3.2mm_M3, F.Cu at (65.8, 30.0)
- added REF**: MountingHole_3.2mm_M3, MountingHole:MountingHole_3.2mm_M3, F.Cu at (65.8, 135.0)
- added REF**: MountingHole_3.2mm_M3, MountingHole:MountingHole_3.2mm_M3, F.Cu at (26.5, 135.0)
- added REF**: MountingHole_3.2mm_M3, MountingHole:MountingHole_3.2mm_M3, F.Cu at (223.2, 135.0)
- added REF**: MountingHole_3.2mm_M3, MountingHole:MountingHole_3.2mm_M3, F.Cu at (144.5, 135.0)
- added REF**: MountingHole_3.2mm_M3, MountingHole:MountingHole_3.2mm_M3, F.Cu at (183.8, 135.0)
- added REF**: MountingHole_3.2mm_M3, MountingHole:MountingHole_3.2mm_M3, F.Cu at (144.5, 30.0)
- added REF**: MountingHole_3.2mm_M3, MountingHole:MountingHole_3.2mm_M3, F.Cu at (105.2, 30.0)
- added REF**: MountingHole_3.2mm_M3, MountingHole:MountingHole_3.2mm_M3, F.Cu at (105.2, 135.0)
- added REF**: MountingHole_3.2mm_M3, MountingHole:MountingHole_3.2mm_M3, F.Cu at (183.8, 30.0)
- added REF**: MountingHole_3.2mm_M3, MountingHole:MountingHole_3.2mm_M3, F.Cu at (262.5, 135.0)
- COL: footprint Connector_PinHeader_2.54mm:PinHeader_1x27_P2.54mm_Vertical -> Connector_PinHeader_2.54mm:PinHeader_1x16_P2.54mm_Vertical
- ROW: footprint Connector_PinHeader_2.54mm:PinHeader_1x12_P2.54mm_Vertical -> Connector_PinHeader_2.54mm:PinHeader_1x08_P2.54mm_Vertical
- moved ROW 13.1 mm to (263.0, 36.0)
Connections:
- COL pad 15: Net-(J1-Pad15) -> GND
- COL pad 16: Net-(J1-Pad16) -> GND
- ROW pad 7: Net-(J2-Pad7) -> GND
- ROW pad 8: Net-(J2-Pad8) -> GND
Other:
- board size 244 x 105.5 mm -> 244 x 113 mm

Commit message: update gerbers
Parts:
- added G***: LOGO, model_d:model_d, B.Cu at (42.5, 37.5)
- added G***: LOGO, model_d:model_d, F.Cu at (42.5, 37.5)
Routing:
- net GND: track 0.00 -> 10.2 mm
